Commit message: kinova arm with camera!

File: kortex_description/arms/gen3_lite/6dof/urdf/gen3_lite_macro.xacro (robot description, xacro)
@@ -3,4 +3,5 @@
   <!-- Propagate last link name information because it is the gripper's parent link -->
   <xacro:property name="last_arm_link" value="dummy_link"/>
+  <xacro:property name="PI" value="3.1415926535897931"/>
   <xacro:macro name="load_arm" params="
     parent
@@ -277,4 +278,27 @@
       <limit lower="0" upper="0" effort="0" velocity="0" />
     </joint>
+    <xacro:if value="${vision}">
+      <!-- sim camera needs to be rotated which might not apply to built in vision module -->
+      <xacro:if value="${sim_gazebo}">
+        <link name="${prefix}camera_link" />
+        <joint name="${prefix}camera_module" type="fixed">
+          <origin xyz="0 0.05639 0.01305" rpy="0 ${-PI/2} ${-PI/2}" />
+          <parent link="${prefix}end_effector_link" />
+          <child  link="${prefix}camera_link" />
+        </joint>
+        <link name="${prefix}camera_depth_frame" />
+        <joint name="${prefix}depth_module" type="fixed">
+          <origin xyz="0.0275 0.066 0.01305" rpy="0 ${-PI/2} ${-PI/2}" />
+          <parent link="${prefix}end_effector_link" />
+          <child  link="${prefix}camera_depth_frame" />
+        </joint>
+        <link name="${prefix}camera_color_frame" />
+        <joint name="${prefix}color_module" type="fixed">
+          <origin xyz="0 0.05639 0.01305" rpy="0 ${-PI/2} ${-PI/2}" />
+          <parent link="${prefix}end_effector_link" />
+          <child  link="${prefix}camera_color_frame" />
+        </joint>
+      </xacro:if>
+    </xacro:if>
   </xacro:macro>
 </robot>

File: kortex_description/grippers/robotiq_2f_140/urdf/robotiq_2f_140_macro.xacro (robot description, xacro)
@@ -26,5 +26,4 @@
         com_port="${com_port}"
         use_fake_hardware="${use_fake_hardware}"
-        mock_sensor_commands="${fake_sensor_commands}"
         sim_gazebo="${sim_gazebo}"
         sim_isaac="${sim_isaac}"

File: kortex_description/grippers/robotiq_2f_85/urdf/robotiq_2f_85_macro.xacro (robot description, xacro)
@@ -26,9 +26,5 @@
         com_port="${com_port}"
         use_fake_hardware="${use_fake_hardware}"
-        mock_sensor_commands="${fake_sensor_commands}"
-        sim_gazebo="${sim_gazebo}"
-        sim_isaac="${sim_isaac}"
-        isaac_joint_commands="${isaac_joint_commands}"
-        isaac_joint_states="${isaac_joint_states}">
+        sim_isaac="${sim_isaac}">
         <origin xyz="0 0 0" rpy="0 0 0" />
     </xacro:robotiq_gripper>

File: kortex_description/robots/kinova.urdf.xacro (robot description, xacro)
@@ -22,9 +22,5 @@
   <xacro:arg name="use_fake_hardware" default="false" />
   <xacro:arg name="fake_sensor_commands" default="false" />
-  <xacro:arg name="sim_gazebo" default="false" />
-  <xacro:arg name="sim_isaac" default="false" />
-  <xacro:arg name="gazebo_renderer" default="ogre"/>
-  <xacro:arg name="camera_width" default="640"/>
-  <xacro:arg name="camera_height" default="480"/>
+  <xacro:arg name="sim_gazebo" default="true" />
   <xacro:arg name="camera_fps" default="6"/>
   <xacro:arg name="simulation_controllers" default="$(find kortex_description)/arm/$(arg arm)/$(arg dof)dof/config/ros2_controllers.yaml" />
@@ -59,5 +55,4 @@
     fake_sensor_commands="$(arg fake_sensor_commands)"
     sim_gazebo="$(arg sim_gazebo)"
-    sim_isaac="$(arg sim_isaac)"
     initial_positions="${xacro.load_yaml(initial_positions_file)}"
     moveit_active="$(arg moveit_active)">
@@ -73,68 +68,43 @@
         <controller_manager_node_name>$(arg prefix)controller_manager</controller_manager_node_name>
       </plugin>
-      <plugin filename="gz-sim-sensors-system" name="gz::sim::systems::Sensors">
-        <render_engine>$(arg gazebo_renderer)</render_engine>
-      </plugin>
     </gazebo>
-    <gazebo reference="camera_color_frame">
-      <sensor name="camera_sensor" type="rgbd_camera">
-        <camera>
-          <horizontal_fov>1.047</horizontal_fov>
-          <image>
-            <width>$(arg camera_width)</width>
-            <height>$(arg camera_height)</height>
-            <format>RGB_INT8</format>
-          </image>
-          <clip>
-            <near>0.1</near>
-            <far>5</far>
-          </clip>
-          <distortion>
-            <k1>0.0</k1>
-            <k2>0.0</k2>
-            <k3>0.0</k3>
-            <p1>0.0</p1>
-            <p2>0.0</p2>
-            <center>0.5 0.5</center>
-          </distortion>
-          <lens>
-            <intrinsics>
-              <fx>554.25469</fx>
-              <fy>554.25469</fy>
-              <cx>320.5</cx>
-              <cy>240.5</cy>
-              <s>0</s>
-            </intrinsics>
-            <!-- These need to match the intrinsics above or
-            Gazebo will default to different default values -->
-            <projection>
-              <p_fx>554.25469</p_fx>
-              <p_fy>554.25469</p_fy>
-              <p_cx>320.5</p_cx>
-              <p_cy>240.5</p_cy>
-              <tx>0</tx>
-              <ty>0</ty>
-            </projection>
-          </lens>
-          <noise>
-            <type>gaussian</type>
-            <mean>0</mean>
-            <stddev>0.00</stddev>
-          </noise>
-          <depth_camera>
+    <gazebo reference="kinova/camera_color_frame">
+      <sensor name="depth_camera" type="depth">
+          <pose>0 0 0 0 0 0</pose>
+          <update_rate>6</update_rate>
+          <camera>
+            <horizontal_fov>1.047</horizontal_fov>
+            <image>
+              <width>640</width>
+              <height>480</height>
+              <format>R8G8B8</format>
+            </image>
             <clip>
-              <near>0.25</near>
-              <far>5</far>
+              <near>0.1</near>
+              <far>10</far>
             </clip>
-          </depth_camera>
-          <optical_frame_id>color_optical_frame</optical_frame_id>
-        </camera>
-        <gz_frame_id>camera_color_frame</gz_frame_id>
-        <always_on>1</always_on>
-        <update_rate>$(arg camera_fps)</update_rate>
-        <visualize>true</visualize>
-        <topic>wrist_mounted_camera</topic>
-        <enable_metrics>false</enable_metrics>
-      </sensor>
+          </camera>
+          <visualize>true</visualize>
+        <topic>kinova/wrist_camera/depth</topic>
+        <enable_metrics>true</enable_metrics>
+        </sensor>
+        <sensor name="rgb_camera" type="camera">
+          <pose>0 0 0 0 0 0</pose>
+          <update_rate>6</update_rate>
+          <camera>
+            <horizontal_fov>1.047</horizontal_fov>
+            <image>
+              <width>640</width>
+              <height>480</height>
+              <format>R8G8B8</format> <!-- or "R8G8B8" for color -->
+            </image>
+            <clip>
+              <near>0.1</near>
+              <far>10</far>
+            </clip>
+          </camera>
+          <topic>kinova/wrist_camera/color</topic>
+        <enable_metrics>true</enable_metrics>
+        </sensor>
     </gazebo>
   </xacro:if>
